Commit message: edited urdf

File: robot_bringup/urdf/cloudy_v2_core.xacro (robot description, xacro)
@@ -37,5 +37,5 @@
             <origin xyz="0 0.15 -0.02" rpy="1.57 0 0"/>
             <geometry>
-                <mesh scale="${scale_ratio} ${scale_ratio} ${scale_ratio}" filename="file://$(find robolaunch_cloudy_description)/urdf/meshes/body_v2.stl"/>
+                <mesh scale="${scale_ratio} ${scale_ratio} ${scale_ratio}" filename="file://$(find robot_bringup)/urdf/meshes/body_v2.stl"/>
             </geometry>
             <material name="gray"/>
@@ -66,5 +66,5 @@
         <visual>
             <geometry>
-                <mesh scale="${scale_ratio} ${scale_ratio} ${scale_ratio}" filename="file://$(find robolaunch_cloudy_description)/urdf/meshes/wheel_v2.stl" />
+                <mesh scale="${scale_ratio} ${scale_ratio} ${scale_ratio}" filename="file://$(find robot_bringup)/urdf/meshes/wheel_v2.stl" />
             </geometry>
             <material name="white"/>
@@ -93,5 +93,5 @@
         <visual>
             <geometry>
-                <mesh scale="${scale_ratio} ${scale_ratio} ${scale_ratio}" filename="file://$(find robolaunch_cloudy_description)/urdf/meshes/wheel_v2.stl" />
+                <mesh scale="${scale_ratio} ${scale_ratio} ${scale_ratio}" filename="file://$(find robot_bringup)/urdf/meshes/wheel_v2.stl" />
             </geometry>
             <origin xyz="-0.067 -0.05 -0.15" rpy="0 0 0" />

File: robot_bringup/urdf/diffbot_system.urdf.xacro (robot description, xacro)
@@ -10,5 +10,5 @@
   <xacro:arg name="prefix" default="" />
   <xacro:arg name="robot_name" default="" />
-  <xacro:include filename="$(find robolaunch_cloudy_description)/urdf/robots/cloudy_v2_core.xacro" />
+  <xacro:include filename="$(find robot_bringup)/urdf/cloudy_v2_core.xacro" />
   <xacro:diffbot prefix="$(arg prefix)"
                   robot_name="$(arg robot_name)"/>

Commit message: update urdf

File: robot_bringup/urdf/cloudy_v2_core.xacro (robot description, xacro)
@@ -21,4 +21,6 @@
     <!-- BASE LINK -->
     <link name="${prefix}base_link">
+    </link>
+    <link name="${prefix}base_footprint">
     </link>
     <joint name="${prefix}base_to_footprint" type="fixed">
